File: power amp/AIA power amp.kicad_pcb (KiCad board)
At the start: 2 copper layers, 27.3 x 39.4 mm, 18 parts, among them J1 AMP POWER, J2 AMP IN, J3 AMP OUT, U1 LM1875

Commit message: Edit amp's feedback compensation cap value
was 150p, now 100p because of availability
Parts:
- C2: value 150p -> 100p
Changed lines of the file:
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@@
       (effects (font (size 1.016 1.016) (thickness 0.2032)))
     )
-    (fp_text value 150p (at -0.635 1.905 180) (layer F.SilkS) hide
+    (fp_text value 100p (at -0.635 1.905 180) (layer F.SilkS) hide
       (effects (font (size 1.016 1.016) (thickness 0.2032)))
     )
