File: power amp/AIA power amp.sch (KiCad schematic (older format))
At the start: 14 parts, among them J1 AMP POWER, J2 AMP IN, J3 AMP OUT, U1 LM1875

Commit message: Edit amp's feedback compensation cap value
was 150p, now 100p because of availability
Parts:
- C2: value 150p -> 100p
Changed lines of the file:
@@
 Sheet 1 1
 Title "AIA Rev. B Power Amp"
-Date "7 mar 2014"
+Date "19 mar 2014"
 Rev "B00"
 Comp "Ali Kocaturk"
@@
 P 3950 2350
 F 0 "C2" H 3950 2450 40  0000 L CNN
-F 1 "150p" H 3956 2265 40  0000 L CNN
+F 1 "100p" H 3956 2265 40  0000 L CNN
 F 2 "~" H 3988 2200 30  0000 C CNN
 F 3 "~" H 3950 2350 60  0000 C CNN
